File: MP6532_board_28-QFN/MP6532_board_28-QFN.kicad_pcb (KiCad board)
At the start: 4 copper layers, 92.5 x 34.6 mm, 78 parts, among them J1 Conn_02x04_Odd_Even, J2 Conn_02x20_Odd_Even, Q1 Q_NMOS_GDS, Q2 Q_NMOS_GDS, Q3 Q_NMOS_GDS, Q4 Q_NMOS_GDS, Q5 Q_NMOS_GDS, Q6 Q_NMOS_GDS, U1 MP6532-QFN, U2 MP6532-ADA-TSOP

Commit message: updated order detail for BDCLC controllers, received working controllers from JLC
Other:
- board text added: "Saitis.net 2025-10-19 v1.2"
- board text removed: "Saitis.net 2025-01-15 v1.1"
