File: MB/MB.kicad_sch (KiCad schematic)
At the start: 93 parts, among them Q1 PNP, Q2 NPN, U1 AM26LV32xD, U2 AM26LV32xD, U3 AM26LV32xD, U4 LM2576HVT-ADJ

Commit message: work on the sensor/legacy barcode scanner connector
Parts:
- added sens2: Conn_01x20_Male, Connector_PinHeader_1.27mm:PinHeader_1x20_P1.27mm_Vertical, symbol Connector:Conn_01x20_Male
Connections:
- net LV32_AinP_Bcode: now reaches sens1.1 (Pin_1)
- net LV32_DinN_Bcode: now reaches sens1.10 (Pin_10)
- net LV32_BinP_Bcode: now reaches sens1.11 (Pin_11)
- net LV32_BinN_Bcode: now reaches sens1.12 (Pin_12)
- net LV32_AinN_Bcode: now reaches sens1.2 (Pin_2)
- net LV31_AoutP_Bcode: now reaches sens1.3 (Pin_3)
- net LV31_AoutN_Bcode: now reaches sens1.4 (Pin_4)
- net LV32_CinP_Bcode: now reaches sens1.5 (Pin_5)
- net LV32_CinN_Bcode: now reaches sens1.6 (Pin_6)
- net LV31_BoutP_Bcode: now reaches sens1.7 (Pin_7)
- net LV31_BoutN_Bcode: now reaches sens1.8 (Pin_8)
- net LV32_DinP_Bcode: now reaches sens1.9 (Pin_9)
- net tape_in_barrier renamed tape_front_present_ir_reflexion
Other:
- note added: "75179B_in"
- note added: "75179B_out"
- note added: "I did no discover that 3 signals from head were driven through differential lines, update in progress Now the rasberry is now on the head of the bot, the idea is to get those now unused barcode readers signals to connect the raspberry pi to the picos running the motors. Also discovered that the connector is crossed between both end: pin 1 = pin 20 at the other end."
- note added: "LV31_Cout"
- note added: "LV31_Dout"
- moved on the sheet: sens1

Commit message: Work on re-using head flat cable, to avoid adding cable between MB and HEAD
Other:
- note added: "A IN 5"
- note added: "A OUT 2 Power +"
- note added: "B IN 6 Serial"
- note added: "B OUT 4 Serial"
- note added: "C OUT 10 Power -"
- note added: "D OUT 3"
- note added: "HEAD Side"
- note added: "I did not discover that 3 signals from head were driven through differential lines, update in progress Now the rasberry is now attached to the head of the bot, the idea is to get those now unused barcode readers signals to connect the raspberry pi to the picos running the motors. Also discovered that the connector is crossed between both ends: pin 1 = pin 20 at the other end. News: the last modif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"
- note added: "IN 7"
- note added: "MB Side"
- note added: "PICO aqui: - 12 quadrants - 2 serial ------------ 16 PICO ctrl: - 6 pwm - 6 dir - 4 mux - 2 analog - 4 serial ---------- 22 MUX 24: in - 6 fault - 3 sensors - vrail - vbat out - 6 sleep - 6 brake"
- note removed: "I did no discover that 3 signals from head were driven through differential lines, update in progress Now the rasberry is now on the head of the bot, the idea is to get those now unused barcode readers signals to connect the raspberry pi to the picos running the motors. Also discovered that the connector is crossed between both end: pin 1 = pin 20 at the other end."
- note removed: "PICO aqui: - 12 quadrants - 4 serial ------------ 16 PICO ctrl: - 6 pwm - 6 dir - 4 mux - 2 analog - 4 serial ---------- 22 MUX 24: in - 6 fault - 3 sensors - vrail - vbat out - 6 sleep - 6 brake"
Changed lines of the file:
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@@
+		)
+	)
+	(text "HEAD Side"
+		(exclude_from_sim no)
+		(at 38.354 113.792 0)
+		(effects
+			(font
+				(size 1.27 1.27)
+			)
+		)
+	)
+	(text "D OUT 3"
+		(exclude_from_sim no)
+		(at 75.692 140.462 0)
+		(effects
+			(font
+				(size 1.27 1.27)
+			)
 		)
 	)
@@
 		)
 	)
-	(text "PICO aqui:\n- 12 quadrants\n- 4 serial\n\n------------\n\n16\n\nPICO ctrl:\n- 6 pwm\n- 6 dir\n- 4 mux\n- 2 analog\n- 4 serial\n\n----------\n\n22\n\n\nMUX 24:\n in\n  - 6 fault\n  - 3 sensors\n  - vrail\n  - vbat\n\n out\n  - 6 sleep\n  - 6 brake\n"
+	(text "PICO aqui:\n- 12 quadrants\n- 2 serial\n\n------------\n\n16\n\nPICO ctrl:\n- 6 pwm\n- 6 dir\n- 4 mux\n- 2 analog\n- 4 serial\n\n----------\n\n22\n\n\nMUX 24:\n in\n  - 6 fault\n  - 3 sensors\n  - vrail\n  - vbat\n\n out\n  - 6 sleep\n  - 6 brake\n"
 		(exclude_from_sim no)
 		(at 15.875 74.295 0)
@@
 		)
 	)
-	(text "I did no discover that 3 signals from head were driven through differential lines,\nupdate in progress\nNow the rasberry is now on the head of the bot, the idea is to get those now\nunused barcode readers signals to connect the raspberry pi to the picos running the motors.\nAlso discovered that the connector is crossed between both end: pin 1 = pin 20 at the other end."
+	(text "B IN 6\nSerial"
 		(exclude_from_sim no)
-		(at 65.024 99.06 0)
+		(at 76.454 135.382 0)
+		(effects
+			(font
+				(size 1.27 1.27)
+			)
+		)
+	)
+	(text "I did not discover that 3 signals from head were driven through differential lines,\nupdate in progress\nNow the rasberry is now attached to the head of the bot, the idea is to get those now\nunused barcode readers signals to connect the raspberry pi to the picos running the motors.\nAlso discovered that the connector is crossed between both ends: pin 1 = pin 20 at the other end.\n\nNews: the last modified bot do not have any additional cable:\n- power is routed via 1,2 and 5,6\n- communication via 7,8 and 11,12"
+		(exclude_from_sim no)
+		(at 61.468 98.552 0)
+		(effects
+			(font
+				(size 1.27 1.27)
+			)
+		)
+	)
+	(text "C OUT 10\nPower -"
+		(exclude_from_sim no)
+		(at 75.692 129.794 0)
+		(effects
+			(font
+				(size 1.27 1.27)
+			)
+		)
+	)
+	(text "IN 7"
+		(exclude_from_sim no)
+		(at 71.882 150.622 0)
+		(effects
+			(font
+				(size 1.27 1.27)
+			)
+		)
+	)
+	(text "A OUT 2\nPower +"
+		(exclude_from_sim no)
+		(at 75.184 120.396 0)
+		(effects
+			(font
+				(size 1.27 1.27)
+			)
+		)
+	)
+	(text "B OUT 4\nSerial"
+		(exclude_from_sim no)
+		(at 75.692 145.034 0)
 		(effects
 			(font
@@
 		(effects
 			(font
+				(size 1.27 1.27)
+			)
+		)
+	)
+	(text "A IN 5"
+		(exclude_from_sim no)
+		(at 74.676 124.968 0)
+		(effects
+			(font
+				(size 1.27 1.27)
+			)
+		)
+	)
+	(text "MB Side"
+		(exclude_from_sim no)
+		(at 56.896 114.046 0)
+		(effects
+			(font

Commit message: PCB calibration marker ready to order
Other:
- note added: "PICO aqui: - 12 quadrants - 2 serial ------------ 14 PICO ctrl: - 6 pwm - 6 dir - 4 mux - 2 analog - 4 serial ---------- 22 MUX 24: in - 6 fault - 3 sensors - vrail - vbat out - 6 sleep - 6 brake"
- note removed: "PICO aqui: - 12 quadrants - 2 serial ------------ 16 PICO ctrl: - 6 pwm - 6 dir - 4 mux - 2 analog - 4 serial ---------- 22 MUX 24: in - 6 fault - 3 sensors - vrail - vbat out - 6 sleep - 6 brake"
Changed lines of the file:
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@@
 		)
 	)
-	(text "PICO aqui:\n- 12 quadrants\n- 2 serial\n\n------------\n\n16\n\nPICO ctrl:\n- 6 pwm\n- 6 dir\n- 4 mux\n- 2 analog\n- 4 serial\n\n----------\n\n22\n\n\nMUX 24:\n in\n  - 6 fault\n  - 3 sensors\n  - vrail\n  - vbat\n\n out\n  - 6 sleep\n  - 6 brake\n"
+	(text "PICO aqui:\n- 12 quadrants\n- 2 serial\n\n------------\n\n14\n\nPICO ctrl:\n- 6 pwm\n- 6 dir\n- 4 mux\n- 2 analog\n- 4 serial\n\n----------\n\n22\n\n\nMUX 24:\n in\n  - 6 fault\n  - 3 sensors\n  - vrail\n  - vbat\n\n out\n  - 6 sleep\n  - 6 brake\n"
 		(exclude_from_sim no)
 		(at 15.875 74.295 0)
