File: 2.5-hdd_box/2.5-hdd_box.kicad_pcb (KiCad board)
At the start: 2 copper layers, 155.9 x 264.2 mm, 41 parts

Commit message: 2.5-hdd_box: cut on bottom for usb-sata board, better placement of soldier pads
Parts:
- moved REF** 3.76 mm to (342.6, 349.8)
- moved REF** 2.80 mm to (283.9, 251.8)
- moved REF** 2.75 mm to (342.6, 251.6)
- moved REF** 2.40 mm to (283.9, 349.8)
- moved REF** 2.16 mm to (252.3, 350.1)
- moved REF** 2.16 mm to (314.0, 251.6)
- moved REF** 1.94 mm to (365.3, 276.3)
- moved REF** 1.84 mm to (342.6, 220.5)
- moved REF** 1.80 mm to (365.2, 324.7)
- moved REF** 1.66 mm to (314.0, 349.8)
- moved REF** 1.51 mm to (283.9, 220.7)
- moved REF** 1.48 mm to (252.3, 220.7)
- moved REF** 1.35 mm to (342.7, 122.2)
- moved REF** 1.10 mm to (252.3, 251.9)
- moved REF** 1.08 mm to (283.9, 122.4)
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Other:
- board size 155.9 x 264.2 mm -> 155.9 x 264.7 mm

Commit message: Cosmetic changes
Other:
- board text added: "T10000/T10K size box for 2.5'' HDD size is not too far from the IBM Jaguar 3592 v0.1"
- board text removed: "T10000/T10K size box for 2.5'' HDD box size is not too far from the IBM jaguar 3592 v0.1"
Changed lines of the file:
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@@
 		)
 	)
-	(gr_text "T10000/T10K size box for 2.5'' HDD box\nsize is not too far from the IBM jaguar 3592\nv0.1\n"
+	(gr_text "T10000/T10K size box for 2.5'' HDD\nsize is not too far from the IBM Jaguar 3592\nv0.1\n"
 		(at 48.1 73.4 0)
 		(layer "Edge.Cuts")

Commit message: height error on side corrected, cosmetics
Parts:
- moved REF** 1.80 mm to (342.7, 92.2)
- moved REF** 1.80 mm to (284.0, 92.3)
- moved REF** 1.80 mm to (314.0, 92.3)
- moved REF** 1.80 mm to (252.4, 92.2)
- moved REF** 1.73 mm to (342.6, 100.3)
- moved REF** 1.50 mm to (252.2, 171.6)
- moved REF** 1.26 mm to (252.3, 100.3)
- moved REF** 1.00 mm to (252.3, 147.3)
- moved REF** 1.00 mm to (252.3, 195.7)
- moved REF** 0.30 mm to (365.6, 195.7)
- moved REF** 0.20 mm to (342.7, 108.3)
- moved REF** 0.20 mm to (283.9, 108.3)
- moved REF** 0.20 mm to (252.5, 108.4)
- moved REF** 0.20 mm to (314.1, 108.3)
- moved REF** 0.10 mm to (365.4, 147.0)
Other:
- board size 155.9 x 264.7 mm -> 155.9 x 266.3 mm

Commit message: last order has small mistakes, this one should be better. Other things added, your responsibility to discover
Parts:
- removed the REF** at (314.0, 349.8)
- added ?: , , F.Cu at (239.0, 152.7)
- added ?: , , F.Cu at (239.0, 240.1)
- added ?: , , F.Cu at (177.6, 240.1)
- added ?: , , F.Cu at (177.6, 152.7)
- added REF**: MountingHole_4.3mm_M4, MountingHole:MountingHole_4.3mm_M4, F.Cu at (177.6, 504.2)
- added REF**: soldpad, Local:soldpad, F.Cu at (193.9, 130.7)
- added REF**: soldpad, Local:soldpad, F.Cu at (194.3, 375.1)
- added REF**: MountingHole_4.3mm_M4, MountingHole:MountingHole_4.3mm_M4, F.Cu at (239.0, 369.5)
- added REF**: MountingHole_4.3mm_M4, MountingHole:MountingHole_4.3mm_M4, F.Cu at (239.0, 504.2)
- added REF**: soldpad, Local:soldpad, F.Cu at (225.4, 115.6)
- added REF**: soldpad, Local:soldpad, F.Cu at (162.6, 130.8)
- added REF**: MountingHole_4.3mm_M4, MountingHole:MountingHole_4.3mm_M4, F.Cu at (177.6, 416.8)
- added REF**: MountingHole_4.3mm_M4, MountingHole:MountingHole_4.3mm_M4, F.Cu at (239.0, 416.8)
- added REF**: soldpad, Local:soldpad, F.Cu at (194.4, 276.5)
- added REF**: MountingHole_4.3mm_M4, MountingHole:MountingHole_4.3mm_M4, F.Cu at (177.6, 369.5)
- added REF**: MountingHole_4.3mm_M4, MountingHole:MountingHole_4.3mm_M4, F.Cu at (239.0, 282.1)
- added REF**: MountingHole_4.3mm_M4, MountingHole:MountingHole_4.3mm_M4, F.Cu at (177.6, 282.1)
- added REF**: soldpad, Local:soldpad, F.Cu at (225.9, 374.9)
- added REF**: soldpad, Local:soldpad, F.Cu at (225.5, 130.7)
- REF** (x6): moved to B.Cu
- moved REF** 124.0 mm to (162.5, 375.1)
- moved REF** 123.8 mm to (162.5, 276.2)
- moved REF** 123.8 mm to (162.4, 115.4), turned to 90 degrees
- moved REF** 122.3 mm to (193.9, 115.6), turned to -90 degrees
- moved REF** 109.1 mm to (177.8, 245.9)
- moved REF** 109.0 mm to (177.8, 133.2)
- moved REF** 108.9 mm to (177.8, 147.1)
- moved REF** 107.0 mm to (239.0, 118.7)
- moved REF** 107.0 mm to (148.8, 118.8)
- moved REF** 106.9 mm to (238.8, 125.8)
- moved REF** 106.6 mm to (261.9, 220.6)
- moved REF** 106.6 mm to (148.6, 220.6)
- moved REF** 106.6 mm to (238.9, 245.4)
- moved REF** 106.6 mm to (148.6, 245.6)
- moved REF** 106.6 mm to (148.7, 147.5)
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Other:
- board size 155.9 x 266.3 mm -> 155.9 x 401 mm
- board text added: "T10000/T10K size box for 2.5'' HDD size is not too far from the IBM Jaguar 3592 v0.2"
- board text added: "Top Cover"
- board text added: "Top strengthener"
- board text added: "What is this crazy Idea to build that witch pcb? - because PCB industry build consistent, reproductible things with a known pipeline - because it's easy to be ul94 - because soldier is better than glue, you can dis-assemble, re-assemble (use a pump to un-glue ;) - giving the SDL of a plastic injection mold, won't really help people - 3D printing does not compete, AFAIK for ul94, reproductibily, e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"
- board text removed: "T10000/T10K size box for 2.5'' HDD size is not too far from the IBM Jaguar 3592 v0.1"
- board text removed: "Top"
